Commit message: Local state

File: bimanual_ws/install/bimanualrobot_description/share/bimanualrobot_description/urdf/control/arm_ros2_controller.urdf.xacro (robot description, xacro)
@@ -1 +1 @@
-/home/thibaut/Documents/Bimanual_Robot/bimanual_ws/src/bimanualrobot_ros2/bimanualrobot_description/urdf/control/arm_ros2_controller.urdf.xacro
+/home/asurite.ad.asu.edu/troisin/Documents/bimanual_mocap/bimanual_ws/src/bimanualrobot_ros2/bimanualrobot_description/urdf/control/arm_ros2_controller.urdf.xacro

File: bimanual_ws/install/bimanualrobot_description/share/bimanualrobot_description/urdf/control/bimanualrobot_ros2_controller.urdf.xacro (robot description, xacro)
@@ -1 +1 @@
-/home/thibaut/Documents/Bimanual_Robot/bimanual_ws/src/bimanualrobot_ros2/bimanualrobot_description/urdf/control/bimanualrobot_ros2_controller.urdf.xacro
+/home/asurite.ad.asu.edu/troisin/Documents/bimanual_mocap/bimanual_ws/src/bimanualrobot_ros2/bimanualrobot_description/urdf/control/bimanualrobot_ros2_controller.urdf.xacro

File: bimanual_ws/install/bimanualrobot_description/share/bimanualrobot_description/urdf/control/common.xacro (robot description, xacro)
@@ -1 +1 @@
-/home/thibaut/Documents/Bimanual_Robot/bimanual_ws/src/bimanualrobot_ros2/bimanualrobot_description/urdf/control/common.xacro
+/home/asurite.ad.asu.edu/troisin/Documents/bimanual_mocap/bimanual_ws/src/bimanualrobot_ros2/bimanualrobot_description/urdf/control/common.xacro

File: bimanual_ws/install/bimanualrobot_description/share/bimanualrobot_description/urdf/control/gazebo_sim_ros2_control.urdf.xacro (robot description, xacro)
@@ -1 +1 @@
-/home/thibaut/Documents/Bimanual_Robot/bimanual_ws/src/bimanualrobot_ros2/bimanualrobot_description/urdf/control/gazebo_sim_ros2_control.urdf.xacro
+/home/asurite.ad.asu.edu/troisin/Documents/bimanual_mocap/bimanual_ws/src/bimanualrobot_ros2/bimanualrobot_description/urdf/control/gazebo_sim_ros2_control.urdf.xacro

File: bimanual_ws/install/bimanualrobot_description/share/bimanualrobot_description/urdf/control/transmission.xacro (robot description, xacro)
@@ -1 +1 @@
-/home/thibaut/Documents/Bimanual_Robot/bimanual_ws/src/bimanualrobot_ros2/bimanualrobot_description/urdf/control/transmission.xacro
+/home/asurite.ad.asu.edu/troisin/Documents/bimanual_mocap/bimanual_ws/src/bimanualrobot_ros2/bimanualrobot_description/urdf/control/transmission.xacro

File: bimanual_ws/install/bimanualrobot_description/share/bimanualrobot_description/urdf/mech/drum.xacro (robot description, xacro)
@@ -1 +1 @@
-/home/thibaut/Documents/Bimanual_Robot/bimanual_ws/src/bimanualrobot_ros2/bimanualrobot_description/urdf/mech/drum.xacro
+/home/asurite.ad.asu.edu/troisin/Documents/bimanual_mocap/bimanual_ws/src/bimanualrobot_ros2/bimanualrobot_description/urdf/mech/drum.xacro

File: bimanual_ws/install/bimanualrobot_description/share/bimanualrobot_description/urdf/mech/drumstick.xacro (robot description, xacro)
@@ -1 +1 @@
-/home/thibaut/Documents/Bimanual_Robot/bimanual_ws/src/bimanualrobot_ros2/bimanualrobot_description/urdf/mech/drumstick.xacro
+/home/asurite.ad.asu.edu/troisin/Documents/bimanual_mocap/bimanual_ws/src/bimanualrobot_ros2/bimanualrobot_description/urdf/mech/drumstick.xacro

File: bimanual_ws/install/bimanualrobot_description/share/bimanualrobot_description/urdf/mech/fingers.xacro (robot description, xacro)
@@ -1 +1 @@
-/home/thibaut/Documents/Bimanual_Robot/bimanual_ws/src/bimanualrobot_ros2/bimanualrobot_description/urdf/mech/fingers.xacro
+/home/asurite.ad.asu.edu/troisin/Documents/bimanual_mocap/bimanual_ws/src/bimanualrobot_ros2/bimanualrobot_description/urdf/mech/fingers.xacro

File: bimanual_ws/install/bimanualrobot_description/share/bimanualrobot_description/urdf/mech/manipulator_h.xacro (robot description, xacro)
@@ -1 +1 @@
-/home/thibaut/Documents/Bimanual_Robot/bimanual_ws/src/bimanualrobot_ros2/bimanualrobot_description/urdf/mech/manipulator_h.xacro
+/home/asurite.ad.asu.edu/troisin/Documents/bimanual_mocap/bimanual_ws/src/bimanualrobot_ros2/bimanualrobot_description/urdf/mech/manipulator_h.xacro

File: bimanual_ws/install/bimanualrobot_description/share/bimanualrobot_description/urdf/mech/manipulator_h_arm.xacro (robot description, xacro)
@@ -1 +1 @@
-/home/thibaut/Documents/Bimanual_Robot/bimanual_ws/src/bimanualrobot_ros2/bimanualrobot_description/urdf/mech/manipulator_h_arm.xacro
+/home/asurite.ad.asu.edu/troisin/Documents/bimanual_mocap/bimanual_ws/src/bimanualrobot_ros2/bimanualrobot_description/urdf/mech/manipulator_h_arm.xacro

File: bimanual_ws/install/bimanualrobot_description/share/bimanualrobot_description/urdf/mech/materials.xacro (robot description, xacro)
@@ -1 +1 @@
-/home/thibaut/Documents/Bimanual_Robot/bimanual_ws/src/bimanualrobot_ros2/bimanualrobot_description/urdf/mech/materials.xacro
+/home/asurite.ad.asu.edu/troisin/Documents/bimanual_mocap/bimanual_ws/src/bimanualrobot_ros2/bimanualrobot_description/urdf/mech/materials.xacro

File: bimanual_ws/install/bimanualrobot_description/share/bimanualrobot_description/urdf/mech/stand.xacro (robot description, xacro)
@@ -1 +1 @@
-/home/thibaut/Documents/Bimanual_Robot/bimanual_ws/src/bimanualrobot_ros2/bimanualrobot_description/urdf/mech/stand.xacro
+/home/asurite.ad.asu.edu/troisin/Documents/bimanual_mocap/bimanual_ws/src/bimanualrobot_ros2/bimanualrobot_description/urdf/mech/stand.xacro

File: bimanual_ws/install/bimanualrobot_description/share/bimanualrobot_description/urdf/robots/bimanual_robot_gazebo.xacro (robot description, xacro)
@@ -1 +1 @@
-/home/thibaut/Documents/Bimanual_Robot/bimanual_ws/src/bimanualrobot_ros2/bimanualrobot_description/urdf/robots/bimanual_robot_gazebo.xacro
+/home/asurite.ad.asu.edu/troisin/Documents/bimanual_mocap/bimanual_ws/src/bimanualrobot_ros2/bimanualrobot_description/urdf/robots/bimanual_robot_gazebo.xacro

File: bimanual_ws/install/bimanualrobot_description/share/bimanualrobot_description/urdf/robots/bimanualrobot.urdf.xacro (robot description, xacro)
@@ -1 +1 @@
-/home/thibaut/Documents/Bimanual_Robot/bimanual_ws/src/bimanualrobot_ros2/bimanualrobot_description/urdf/robots/bimanualrobot.urdf.xacro
+/home/asurite.ad.asu.edu/troisin/Documents/bimanual_mocap/bimanual_ws/src/bimanualrobot_ros2/bimanualrobot_description/urdf/robots/bimanualrobot.urdf.xacro

File: bimanual_ws/install/bimanualrobot_drumstick_moveit_config/share/bimanualrobot_drumstick_moveit_config/config/bimanualrobot.ros2_control.xacro (robot description, xacro)
@@ -1 +1 @@
-/home/thibaut/Documents/Bimanual_Robot/bimanual_ws/src/bimanualrobot_ros2/bimanualrobot_drumstick_moveit_config/config/bimanualrobot.ros2_control.xacro
+/home/asurite.ad.asu.edu/troisin/Documents/bimanual_mocap/bimanual_ws/src/bimanualrobot_ros2/bimanualrobot_drumstick_moveit_config/config/bimanualrobot.ros2_control.xacro

File: bimanual_ws/install/bimanualrobot_drumstick_moveit_config/share/bimanualrobot_drumstick_moveit_config/config/bimanualrobot.urdf.xacro (robot description, xacro)
@@ -1 +1 @@
-/home/thibaut/Documents/Bimanual_Robot/bimanual_ws/src/bimanualrobot_ros2/bimanualrobot_drumstick_moveit_config/config/bimanualrobot.urdf.xacro
+/home/asurite.ad.asu.edu/troisin/Documents/bimanual_mocap/bimanual_ws/src/bimanualrobot_ros2/bimanualrobot_drumstick_moveit_config/config/bimanualrobot.urdf.xacro

File: bimanual_ws/src/bimanualrobot_ros2/bimanualrobot_description/urdf/robots/bimanualrobot.urdf (robot description, URDF)
Before this commit: robot bimanualrobot, 19 links, 18 joints
Links:
- link leftarm_forearm_link: geometry collision mesh filename=/home/asurite.ad.asu.edu/troisin/Documents/bimanual_mocap/b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; visual mesh filename=/home/asurite.ad.asu.edu/troisin/Documents/bimanual_mocap/b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 scale=0.001 0.001 0.001
- link leftarm_shoulder_link: geometry collision box size=0.054 0.054 0.126; visual mesh filename=/home/asurite.ad.asu.edu/troisin/Documents/bimanual_mocap/b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 scale=0.001 0.001 0.001
- link leftarm_upper_arm_link: geometry collision box size=0.06 0.14 0.06; visual mesh filename=/home/asurite.ad.asu.edu/troisin/Documents/bimanual_mocap/b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 scale=0.001 0.001 0.001
- link leftarm_wrist_1_link: geometry collision mesh filename=/home/asurite.ad.asu.edu/troisin/Documents/bimanual_mocap/b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; visual mesh filename=/home/asurite.ad.asu.edu/troisin/Documents/bimanual_mocap/b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 scale=0.001 0.001 0.001
- link leftarm_wrist_2_link: geometry collision box size=0.048 0.09 0.048; visual mesh filename=/home/asurite.ad.asu.edu/troisin/Documents/bimanual_mocap/b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 scale=0.001 0.001 0.001
- link leftarm_wrist_3_link: geometry collision mesh filename=/home/asurite.ad.asu.edu/troisin/Documents/bimanual_mocap/b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; visual mesh filename=/home/asurite.ad.asu.edu/troisin/Documents/bimanual_mocap/b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 scale=0.001 0.001 0.001
- link rightarm_forearm_link: geometry collision mesh filename=/home/asurite.ad.asu.edu/troisin/Documents/bimanual_mocap/b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; visual mesh filename=/home/asurite.ad.asu.edu/troisin/Documents/bimanual_mocap/b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 scale=0.001 0.001 0.001
- link rightarm_shoulder_link: geometry collision box size=0.054 0.054 0.126; visual mesh filename=/home/asurite.ad.asu.edu/troisin/Documents/bimanual_mocap/b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 scale=0.001 0.001 0.001
- link rightarm_upper_arm_link: geometry collision box size=0.06 0.14 0.06; visual mesh filename=/home/asurite.ad.asu.edu/troisin/Documents/bimanual_mocap/b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 scale=0.001 0.001 0.001
- link rightarm_wrist_1_link: geometry collision mesh filename=/home/asurite.ad.asu.edu/troisin/Documents/bimanual_mocap/b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; visual mesh filename=/home/asurite.ad.asu.edu/troisin/Documents/bimanual_mocap/b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 scale=0.001 0.001 0.001
- link rightarm_wrist_2_link: geometry collision box size=0.048 0.09 0.048; visual mesh filename=/home/asurite.ad.asu.edu/troisin/Documents/bimanual_mocap/b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 scale=0.001 0.001 0.001
- link rightarm_wrist_3_link: geometry collision mesh filename=/home/asurite.ad.asu.edu/troisin/Documents/bimanual_mocap/b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; visual mesh filename=/home/asurite.ad.asu.edu/troisin/Documents/bimanual_mocap/b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 scale=0.001 0.001 0.001
- link stand_link: geometry collision mesh filename=/home/asurite.ad.asu.edu/troisin/Documents/bimanual_mocap/b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; visual mesh filename=/home/asurite.ad.asu.edu/troisin/Documents/bimanual_mocap/b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

File: bimanual_ws/src/bimanualrobot_ros2/bimanualrobot_description/urdf/robots/bimanualrobot.urdf.xacro (robot description, xacro)
@@ -10,5 +10,5 @@
   <xacro:arg name="use_gazebo" default="false"/>
   <xacro:arg name="use_gripper" default="false"/>
-  <xacro:arg name="use_drumstick" default="false"/>
+  <xacro:arg name="use_drumstick" default="true"/>
   <xacro:property name="gripper_type" value="$(arg gripper_type)"/>
   <!-- manipulator_h arm-->
@@ -24,5 +24,5 @@
   <!-- drumstick -->
   <xacro:if value="$(arg use_drumstick)">
-    <xacro:include filename="$(find bimanualrobot_description)/urdf/mech/drumstick.xacro" />
+    <xacro:include filename="$(find bimanualrobot_description)/urdf/mech/pingpong.xacro" />
     <xacro:include filename="$(find bimanualrobot_description)/urdf/mech/drum.xacro" />
   </xacro:if>
@@ -87,10 +87,10 @@
   </joint>
   <xacro:if value="$(arg use_drumstick)">
-    <xacro:drumstick prefix="leftarm" parent="leftarm_ee_link">
+    <xacro:ping prefix="leftarm" parent="leftarm_ee_link">
       <origin xyz="0 0 0.086" rpy="0 0 0" />
-    </xacro:drumstick>
-    <xacro:drumstick prefix="rightarm" parent="rightarm_ee_link">
+    </xacro:ping>
+    <xacro:ping prefix="rightarm" parent="rightarm_ee_link">
       <origin xyz="0 0 0.086" rpy="0 0 0" />
-    </xacro:drumstick>
+    </xacro:ping>
   </xacro:if>
   <xacro:include filename="$(find bimanualrobot_description)/urdf/control/gazebo_sim_ros2_control.urdf.xacro" />
