Commit message: world

File: bimanual_ws/src/bimanualrobot_ros2/bimanualrobot_description/urdf/robots/bimanualrobot.urdf (robot description, URDF)
Before this commit: robot bimanualrobot, 19 links, 18 joints
Links:
- link leftarm_forearm_link: geometry collision mesh filename=/home/thibaut/Documents/bimanual_mocap/bimanual_ws/src/bima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; visual mesh filename=/home/thibaut/Documents/bimanual_mocap/bimanual_ws/src/bima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 scale=0.001 0.001 0.001
- link leftarm_shoulder_link: geometry collision box size=0.054 0.054 0.126; visual mesh filename=/home/thibaut/Documents/bimanual_mocap/bimanual_ws/src/bima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 scale=0.001 0.001 0.001
- link leftarm_upper_arm_link: geometry collision box size=0.06 0.14 0.06; visual mesh filename=/home/thibaut/Documents/bimanual_mocap/bimanual_ws/src/bima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 scale=0.001 0.001 0.001
- link leftarm_wrist_1_link: geometry collision mesh filename=/home/thibaut/Documents/bimanual_mocap/bimanual_ws/src/bima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; visual mesh filename=/home/thibaut/Documents/bimanual_mocap/bimanual_ws/src/bima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 scale=0.001 0.001 0.001
- link leftarm_wrist_2_link: geometry collision box size=0.048 0.09 0.048; visual mesh filename=/home/thibaut/Documents/bimanual_mocap/bimanual_ws/src/bima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 scale=0.001 0.001 0.001
- link leftarm_wrist_3_link: geometry collision mesh filename=/home/thibaut/Documents/bimanual_mocap/bimanual_ws/src/bima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; visual mesh filename=/home/thibaut/Documents/bimanual_mocap/bimanual_ws/src/bima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 scale=0.001 0.001 0.001
- link rightarm_forearm_link: geometry collision mesh filename=/home/thibaut/Documents/bimanual_mocap/bimanual_ws/src/bima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; visual mesh filename=/home/thibaut/Documents/bimanual_mocap/bimanual_ws/src/bima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 scale=0.001 0.001 0.001
- link rightarm_shoulder_link: geometry collision box size=0.054 0.054 0.126; visual mesh filename=/home/thibaut/Documents/bimanual_mocap/bimanual_ws/src/bima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 scale=0.001 0.001 0.001
- link rightarm_upper_arm_link: geometry collision box size=0.06 0.14 0.06; visual mesh filename=/home/thibaut/Documents/bimanual_mocap/bimanual_ws/src/bima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 scale=0.001 0.001 0.001
- link rightarm_wrist_1_link: geometry collision mesh filename=/home/thibaut/Documents/bimanual_mocap/bimanual_ws/src/bima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; visual mesh filename=/home/thibaut/Documents/bimanual_mocap/bimanual_ws/src/bima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 scale=0.001 0.001 0.001
- link rightarm_wrist_2_link: geometry collision box size=0.048 0.09 0.048; visual mesh filename=/home/thibaut/Documents/bimanual_mocap/bimanual_ws/src/bima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 scale=0.001 0.001 0.001
- link rightarm_wrist_3_link: geometry collision mesh filename=/home/thibaut/Documents/bimanual_mocap/bimanual_ws/src/bima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; visual mesh filename=/home/thibaut/Documents/bimanual_mocap/bimanual_ws/src/bima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 scale=0.001 0.001 0.001
- link stand_link: geometry collision mesh filename=/home/thibaut/Documents/bimanual_mocap/bimanual_ws/src/bima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; visual mesh filename=/home/thibaut/Documents/bimanual_mocap/bimanual_ws/src/bima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

Commit message: Reset repo to local state

File: bimanual_ws/src/bimanualrobot_ros2/bimanualrobot_description/urdf/robots/bimanualrobot.urdf (robot description, URDF)
Before this commit: robot bimanualrobot, 19 links, 18 joints
Links:
- added link leftarm_racket_blade, mass 0.12; collision cylinder length=0.02 radius=0.095; visual cylinder length=0.02 radius=0.095
- added link leftarm_racket_handle, mass 0.05; collision box size=0.028 0.022 0.14; visual box size=0.028 0.022 0.14
- added link rightarm_racket_blade, mass 0.12; collision cylinder length=0.02 radius=0.095; visual cylinder length=0.02 radius=0.095
- added link rightarm_racket_handle, mass 0.05; collision box size=0.028 0.022 0.14; visual box size=0.028 0.022 0.14
- link leftarm_forearm_link: geometry collision mesh filename=file:///home/thibaut/Documents/bimanual_mocap/bimanual_ws/i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; visual mesh filename=file:///home/thibaut/Documents/bimanual_mocap/bimanual_ws/i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 scale=0.001 0.001 0.001
- link leftarm_shoulder_link: geometry collision box size=0.054 0.054 0.126; visual mesh filename=file:///home/thibaut/Documents/bimanual_mocap/bimanual_ws/i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 scale=0.001 0.001 0.001
- link leftarm_upper_arm_link: geometry collision box size=0.06 0.14 0.06; visual mesh filename=file:///home/thibaut/Documents/bimanual_mocap/bimanual_ws/i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 scale=0.001 0.001 0.001
- link leftarm_wrist_1_link: geometry collision mesh filename=file:///home/thibaut/Documents/bimanual_mocap/bimanual_ws/i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; visual mesh filename=file:///home/thibaut/Documents/bimanual_mocap/bimanual_ws/i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 scale=0.001 0.001 0.001
- link leftarm_wrist_2_link: geometry collision box size=0.048 0.09 0.048; visual mesh filename=file:///home/thibaut/Documents/bimanual_mocap/bimanual_ws/i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 scale=0.001 0.001 0.001
- link leftarm_wrist_3_link: geometry collision mesh filename=file:///home/thibaut/Documents/bimanual_mocap/bimanual_ws/i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; visual mesh filename=file:///home/thibaut/Documents/bimanual_mocap/bimanual_ws/i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 scale=0.001 0.001 0.001
- link rightarm_forearm_link: geometry collision mesh filename=file:///home/thibaut/Documents/bimanual_mocap/bimanual_ws/i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; visual mesh filename=file:///home/thibaut/Documents/bimanual_mocap/bimanual_ws/i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 scale=0.001 0.001 0.001
- link rightarm_shoulder_link: geometry collision box size=0.054 0.054 0.126; visual mesh filename=file:///home/thibaut/Documents/bimanual_mocap/bimanual_ws/i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 scale=0.001 0.001 0.001
- link rightarm_upper_arm_link: geometry collision box size=0.06 0.14 0.06; visual mesh filename=file:///home/thibaut/Documents/bimanual_mocap/bimanual_ws/i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 scale=0.001 0.001 0.001
- link rightarm_wrist_1_link: geometry collision mesh filename=file:///home/thibaut/Documents/bimanual_mocap/bimanual_ws/i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; visual mesh filename=file:///home/thibaut/Documents/bimanual_mocap/bimanual_ws/i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 scale=0.001 0.001 0.001
- link rightarm_wrist_2_link: geometry collision box size=0.048 0.09 0.048; visual mesh filename=file:///home/thibaut/Documents/bimanual_mocap/bimanual_ws/i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 scale=0.001 0.001 0.001
- link rightarm_wrist_3_link: geometry collision mesh filename=file:///home/thibaut/Documents/bimanual_mocap/bimanual_ws/i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; visual mesh filename=file:///home/thibaut/Documents/bimanual_mocap/bimanual_ws/i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 scale=0.001 0.001 0.001
- link stand_link: geometry collision mesh filename=file:///home/thibaut/Documents/bimanual_mocap/bimanual_ws/i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; visual mesh filename=file:///home/thibaut/Documents/bimanual_mocap/bimanual_ws/i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
Joints:
- added joint leftarm_racket_handle_joint: type fixed, parent leftarm_racket_handle, child leftarm_racket_blade, origin xyz=0 0 0.0945 rpy=0 0 0
- added joint leftarm_racket_mount_joint: type fixed, parent leftarm_ee_link, child leftarm_racket_handle, origin xyz=0 0 0.086 rpy=0 0 0
- added joint rightarm_racket_handle_joint: type fixed, parent rightarm_racket_handle, child rightarm_racket_blade, origin xyz=0 0 0.0945 rpy=0 0 0
- added joint rightarm_racket_mount_joint: type fixed, parent rightarm_ee_link, child rightarm_racket_handle, origin xyz=0 0 0.086 rpy=0 0 0
- joint leftarm_elbow_joint: limit lower=-1.2566370614359172 upper=2.261946710584651 effort=1000 velocity=15 -> lower=-1.2566370614359172 upper=2.261946710584651 effort=250 velocity=6.5
- joint leftarm_shoulder_lift_joint: limit lower=-1.7803405567893358 upper=1.7803405567893358 effort=1000 velocity=15 -> lower=-1.7803405567893358 upper=1.7803405567893358 effort=250 velocity=6.5
- joint leftarm_shoulder_pan_joint: limit lower=-3.141592653589793 upper=0 effort=1000 velocity=15 -> lower=-3.141592653589793 upper=0 effort=250 velocity=6.5
- joint leftarm_wrist_1_joint: limit lower=-3.141592653589793 upper=3.141592653589793 effort=1000 velocity=15 -> lower=-3.141592653589793 upper=3.141592653589793 effort=250 velocity=6.5
- joint leftarm_wrist_2_joint: limit lower=-1.5707963267948966 upper=1.5707963267948966 effort=1000 velocity=15 -> lower=-1.5707963267948966 upper=1.5707963267948966 effort=250 velocity=6.5
- joint leftarm_wrist_3_joint: limit lower=-3.141592653589793 upper=3.141592653589793 effort=1000 velocity=15 -> lower=-3.141592653589793 upper=3.141592653589793 effort=250 velocity=6.5
- joint rightarm_elbow_joint: limit lower=-1.2566370614359172 upper=2.261946710584651 effort=1000 velocity=15 -> lower=-1.2566370614359172 upper=2.261946710584651 effort=250 velocity=6.5
- joint rightarm_shoulder_lift_joint: limit lower=-1.7803405567893358 upper=1.7803405567893358 effort=1000 velocity=15 -> lower=-1.7803405567893358 upper=1.7803405567893358 effort=250 velocity=6.5
- joint rightarm_shoulder_pan_joint: limit lower=0 upper=3.141592653589793 effort=1000 velocity=15 -> lower=0 upper=3.141592653589793 effort=250 velocity=6.5
- joint rightarm_wrist_1_joint: limit lower=-3.141592653589793 upper=3.141592653589793 effort=1000 velocity=15 -> lower=-3.141592653589793 upper=3.141592653589793 effort=250 velocity=6.5
- joint rightarm_wrist_2_joint: limit lower=-1.5707963267948966 upper=1.5707963267948966 effort=1000 velocity=15 -> lower=-1.5707963267948966 upper=1.5707963267948966 effort=250 velocity=6.5
- joint rightarm_wrist_3_joint: limit lower=-3.141592653589793 upper=3.141592653589793 effort=1000 velocity=15 -> lower=-3.141592653589793 upper=3.141592653589793 effort=250 velocity=6.5

File: bimanual_ws/src/bimanualrobot_ros2/bimanualrobot_description/urdf/robots/bimanualrobot.urdf.xacro (robot description, xacro)
@@ -10,5 +10,5 @@
   <xacro:arg name="use_gazebo" default="false"/>
   <xacro:arg name="use_gripper" default="false"/>
-  <xacro:arg name="use_drumstick" default="true"/>
+  <xacro:arg name="use_cup_and_ball" default="true"/>
   <xacro:property name="gripper_type" value="$(arg gripper_type)"/>
   <!-- manipulator_h arm-->
@@ -22,8 +22,7 @@
     </xacro:if>
   </xacro:if>
-  <!-- drumstick -->
-  <xacro:if value="$(arg use_drumstick)">
-    <xacro:include filename="$(find bimanualrobot_description)/urdf/mech/pingpong.xacro" />
-    <xacro:include filename="$(find bimanualrobot_description)/urdf/mech/drum.xacro" />
+  <!-- cup and ball -->
+  <xacro:if value="$(arg use_cup_and_ball)">
+    <xacro:include filename="$(find bimanualrobot_description)/urdf/mech/cup_and_ball.xacro" />
   </xacro:if>
   <link name="base_link"/>
@@ -86,11 +85,13 @@
     <origin xyz="0 0 0" rpy="0 0 0" />
   </joint>
-  <xacro:if value="$(arg use_drumstick)">
-    <xacro:ping prefix="leftarm" parent="leftarm_ee_link">
-      <origin xyz="0 0 0.086" rpy="0 0 0" />
-    </xacro:ping>
-    <xacro:ping prefix="rightarm" parent="rightarm_ee_link">
-      <origin xyz="0 0 0.086" rpy="0 0 0" />
-    </xacro:ping>
+  <xacro:if value="$(arg use_cup_and_ball)">
+    <!-- Left cup and ball - matching MuJoCo orientation (1.5707963 0 0) -->
+    <xacro:cup_and_ball prefix="leftarm" parent="leftarm_ee_link">
+      <origin xyz="0 0.15 0.09" rpy="1.5707963 0 0" />
+    </xacro:cup_and_ball>
+    <!-- Right cup and ball - ADD PI rotation to compensate for arm orientation difference -->
+    <xacro:cup_and_ball prefix="rightarm" parent="rightarm_ee_link">
+      <origin xyz="0 -0.15 0.09" rpy="1.5707963 0 ${pi}" />
+    </xacro:cup_and_ball>
   </xacro:if>
   <xacro:include filename="$(find bimanualrobot_description)/urdf/control/gazebo_sim_ros2_control.urdf.xacro" />
@@ -116,16 +117,16 @@
   <xacro:arg name="ball_rpy" default="0 0 0"/>
   <xacro:if value="$(arg show_ball_ref)">
-    <link name="pingpong_ref_link">
+    <link name="ball_ref_link">
       <visual>
         <origin xyz="$(arg ball_xyz)" rpy="$(arg ball_rpy)"/>
-        <geometry><sphere radius="0.02"/></geometry>
-        <material name="White">
-          <color rgba="1 1 1 1"/>
+        <geometry><sphere radius="0.04"/></geometry>
+        <material name="Orange">
+          <color rgba="1 0.5 0 0.5"/>
         </material>
       </visual>
     </link>
-    <joint name="world_to_pingpong_ref" type="fixed">
+    <joint name="world_to_ball_ref" type="fixed">
       <parent link="world"/>
-      <child link="pingpong_ref_link"/>
+      <child link="ball_ref_link"/>
       <origin xyz="0 0 0" rpy="0 0 0"/>
     </joint>
