Commit message: final

File: bimanual_ws/src/bimanualrobot_ros2/bimanualrobot_description/urdf/control/arm_ros2_controller.urdf.xacro (robot description, xacro)
@@ -108,5 +108,5 @@
         <param name="Torque Enable">1</param>
         <param name="Operating Mode">3</param>
-        <param name="Position P Gain">10</param>
+        <param name="Position P Gain">13</param>
         <param name="Return Delay Time">0</param>
       </gpio>
@@ -123,5 +123,5 @@
         <param name="Torque Enable">1</param>
         <param name="Operating Mode">3</param>
-        <param name="Position P Gain">10</param>
+        <param name="Position P Gain">13</param>
         <param name="Return Delay Time">0</param>
       </gpio>
@@ -138,5 +138,5 @@
         <param name="Torque Enable">1</param>
         <param name="Operating Mode">3</param>
-        <param name="Position P Gain">10</param>
+        <param name="Position P Gain">13</param>
         <param name="Return Delay Time">0</param>
       </gpio>
@@ -153,5 +153,5 @@
         <param name="Torque Enable">1</param>
         <param name="Operating Mode">3</param>
-        <param name="Position P Gain">10</param>
+        <param name="Position P Gain">13</param>
         <param name="Return Delay Time">0</param>
       </gpio>
@@ -168,5 +168,5 @@
         <param name="Torque Enable">1</param>
         <param name="Operating Mode">3</param>
-        <param name="Position P Gain">10</param>
+        <param name="Position P Gain">13</param>
         <param name="Return Delay Time">0</param>
       </gpio>
@@ -183,5 +183,5 @@
         <param name="Torque Enable">1</param>
         <param name="Operating Mode">3</param>
-        <param name="Position P Gain">10</param>
+        <param name="Position P Gain">13</param>
         <param name="Return Delay Time">0</param>
       </gpio>
