Commit message: final

File: bimanual_ws/src/bimanualrobot_ros2/bimanualrobot_description/urdf/mech/cup_and_ball.xacro (robot description, xacro)
@@ -1,175 +1,236 @@
 <?xml version="1.0"?>
 <robot xmlns:xacro="http://www.ros.org/wiki/xacro">
-  <xacro:macro name="cup_and_ball" params="prefix parent *origin">
-    <!-- Cup pole (small cylinder under the cup) -->
-    <link name="${prefix}_cup_pole">
+  <!--
+    cup_and_ball macro
+    params:
+      prefix      : "left" or "right"
+      parent      : parent link name
+      z_dir       : 1 for left cup (pole below, opening above),
+                   -1 for right cup (pole above, opening below)
+      seg_rgba    : RGBA string for the 32 wall segments
+      sensor_rgba : RGBA string for the sensor disc
+      *origin     : joint origin block (position/orientation of cup relative to parent)
+  -->
+  <xacro:macro name="cup_and_ball"
+               params="prefix parent z_dir:=1
+                       seg_rgba:='0.165 0.741 0.894 1'
+                       sensor_rgba:='0.165 0.741 0.894 0.3'
+                       *origin">
+    <!-- Single rigid link holds all cup geometry (matches MuJoCo single body) -->
+    <link name="${prefix}_cup">
+      <!-- Approximate inertia for the cup assembly (mass=0.08) -->
+      <inertial>
+        <origin xyz="0 0 ${z_dir * 0.03}" rpy="0 0 0"/>
+        <mass value="0.08"/>
+        <inertia ixx="0.0005" ixy="0.0" ixz="0.0"
+                 iyy="0.0005" iyz="0.0"
+                 izz="0.0005"/>
+      </inertial>
+      <!-- ── Small pole under/over the cup ─────────────────────────────────── -->
+      <!--   MuJoCo: cylinder size="0.0075 0.04"  (radius half-length)         -->
+      <!--   URDF  : radius=0.0075  length=0.08                                -->
       <visual>
-        <origin xyz="0 0 0.04" rpy="0 0 0"/>
-        <geometry>
-          <cylinder radius="0.0075" length="0.08"/>
-        </geometry>
+        <origin xyz="0 0 ${z_dir * -0.04}" rpy="0 0 0"/>
+        <geometry><cylinder radius="0.0075" length="0.08"/></geometry>
         <material name="wood"/>
       </visual>
       <collision>
-        <origin xyz="0 0 0.04" rpy="0 0 0"/>
-        <geometry>
-          <cylinder radius="0.0075" length="0.08"/>
-        </geometry>
+        <origin xyz="0 0 ${z_dir * -0.04}" rpy="0 0 0"/>
+        <geometry><cylinder radius="0.0075" length="0.08"/></geometry>
       </collision>
-      <inertial>
-        <origin xyz="0 0 0.04" rpy="0 0 0"/>
-        <mass value="0.005"/>
-        <inertia ixx="0.00001" ixy="0.0" ixz="0.0"
-                 iyy="0.00001" iyz="0.0"
-                 izz="0.000001"/>
-      </inertial>
-    </link>
-    <!-- Cup bottom (flat cylinder) -->
-    <link name="${prefix}_cup_bottom">
+      <!-- ── Cup bottom (wide flat cylinder) ───────────────────────────────── -->
+      <!--   radius=0.085 (scaled ×0.85 from original 0.1)  length=0.1          -->
       <visual>
-        <origin xyz="0 0 0" rpy="0 0 0"/>
-        <geometry>
-          <cylinder radius="0.05" length="0.01"/>
-        </geometry>
-        <material name="wood"/>
+        <origin xyz="0 0 ${z_dir * -0.01}" rpy="0 0 0"/>
+        <geometry><cylinder radius="0.085" length="0.1"/></geometry>
+        <material name="wood">
+          <color rgba="0.4 0.4 0.4 1"/>
+        </material>
       </visual>
       <collision>
-        <origin xyz="0 0 0" rpy="0 0 0"/>
-        <geometry>
-          <cylinder radius="0.1" length="0.01"/>
-        </geometry>
+        <origin xyz="0 0 ${z_dir * -0.01}" rpy="0 0 0"/>
+        <geometry><cylinder radius="0.085" length="0.1"/></geometry>
       </collision>
-      <inertial>
-        <origin xyz="0 0 0" rpy="0 0 0"/>
-        <mass value="0.02"/>
-        <inertia ixx="0.0001" ixy="0.0" ixz="0.0"
-                 iyy="0.0001" iyz="0.0"
-                 izz="0.0002"/>
-      </inertial>
-    </link>
-    <!-- Cup wall +X -->
-    <link name="${prefix}_cup_wall_x_plus">
+      <!-- ── Sensor disc (thin cylinder) ───────────────────────────────────── -->
+      <!--   radius=0.077 (scaled ×0.85 from original 0.09)  length=0.02        -->
       <visual>
-        <origin xyz="0 0 0" rpy="0 0 0"/>
-        <geometry>
-          <box size="0.005 0.1 0.1"/>
-        </geometry>
-        <material name="wood"/>
+        <origin xyz="0 0 ${z_dir * 0.02}" rpy="0 0 0"/>
+        <geometry><cylinder radius="0.077" length="0.02"/></geometry>
+        <material name="${prefix}_sensor_mat">
+          <color rgba="${sensor_rgba}"/>
+        </material>
       </visual>
       <collision>
-        <origin xyz="0 0 0" rpy="0 0 0"/>
-        <geometry>
-          <box size="0.005 0.1 0.1"/>
-        </geometry>
+        <origin xyz="0 0 ${z_dir * 0.02}" rpy="0 0 0"/>
+        <geometry><cylinder radius="0.077" length="0.02"/></geometry>
       </collision>
-      <inertial>
-        <origin xyz="0 0 0" rpy="0 0 0"/>
-        <mass value="0.015"/>
-        <inertia ixx="0.0001" ixy="0.0" ixz="0.0"
-                 iyy="0.0001" iyz="0.0"
-                 izz="0.00001"/>
-      </inertial>
+      <!-- ── 32 wall segments ───────────────────────────────────────────────── -->
+      <!--   x/y positions scaled ×0.85 from original (radius ~0.1044 → ~0.0888) -->
+      <visual><origin xyz="0.088820 0.008748 ${z_dir * 0.03}" rpy="0 0 0.098175"/>
+        <geometry><box size="0.01 0.020616 0.2"/></geometry>
+        <material name="${prefix}_seg_mat"><color rgba="${seg_rgba}"/></material></visual>
+      <collision><origin xyz="0.088820 0.008748 ${z_dir * 0.03}" rpy="0 0 0.098175"/>
+        <geometry><box size="0.01 0.020616 0.2"/></geometry></collision>
+      <visual><origin xyz="0.085407 0.025908 ${z_dir * 0.03}" rpy="0 0 0.294524"/>
+        <geometry><box size="0.01 0.020616 0.2"/></geometry>
+        <material name="${prefix}_seg_mat"><color rgba="${seg_rgba}"/></material></visual>
+      <collision><origin xyz="0.085407 0.025908 ${z_dir * 0.03}" rpy="0 0 0.294524"/>
+        <geometry><box size="0.01 0.020616 0.2"/></geometry></collision>
+      <visual><origin xyz="0.078712 0.042072 ${z_dir * 0.03}" rpy="0 0 0.490874"/>
+        <geometry><box size="0.01 0.020616 0.2"/></geometry>
+        <material name="${prefix}_seg_mat"><color rgba="${seg_rgba}"/></material></visual>
+      <collision><origin xyz="0.078712 0.042072 ${z_dir * 0.03}" rpy="0 0 0.490874"/>
+        <geometry><box size="0.01 0.020616 0.2"/></geometry></collision>
+      <visual><origin xyz="0.068991 0.056619 ${z_dir * 0.03}" rpy="0 0 0.687223"/>
+        <geometry><box size="0.01 0.020616 0.2"/></geometry>
+        <material name="${prefix}_seg_mat"><color rgba="${seg_rgba}"/></material></visual>
+      <collision><origin xyz="0.068991 0.056619 ${z_dir * 0.03}" rpy="0 0 0.687223"/>
+        <geometry><box size="0.01 0.020616 0.2"/></geometry></collision>
+      <visual><origin xyz="0.056619 0.068991 ${z_dir * 0.03}" rpy="0 0 0.883573"/>
+        <geometry><box size="0.01 0.020616 0.2"/></geometry>
+        <material name="${prefix}_seg_mat"><color rgba="${seg_rgba}"/></material></visual>
+      <collision><origin xyz="0.056619 0.068991 ${z_dir * 0.03}" rpy="0 0 0.883573"/>
+        <geometry><box size="0.01 0.020616 0.2"/></geometry></collision>
+      <visual><origin xyz="0.042072 0.078712 ${z_dir * 0.03}" rpy="0 0 1.079922"/>
+        <geometry><box size="0.01 0.020616 0.2"/></geometry>
+        <material name="${prefix}_seg_mat"><color rgba="${seg_rgba}"/></material></visual>
+      <collision><origin xyz="0.042072 0.078712 ${z_dir * 0.03}" rpy="0 0 1.079922"/>
+        <geometry><box size="0.01 0.020616 0.2"/></geometry></collision>
+      <visual><origin xyz="0.025908 0.085407 ${z_dir * 0.03}" rpy="0 0 1.276272"/>
+        <geometry><box size="0.01 0.020616 0.2"/></geometry>
+        <material name="${prefix}_seg_mat"><color rgba="${seg_rgba}"/></material></visual>
+      <collision><origin xyz="0.025908 0.085407 ${z_dir * 0.03}" rpy="0 0 1.276272"/>
+        <geometry><box size="0.01 0.020616 0.2"/></geometry></collision>
+      <visual><origin xyz="0.008748 0.088820 ${z_dir * 0.03}" rpy="0 0 1.472622"/>
+        <geometry><box size="0.01 0.020616 0.2"/></geometry>
+        <material name="${prefix}_seg_mat"><color rgba="${seg_rgba}"/></material></visual>
+      <collision><origin xyz="0.008748 0.088820 ${z_dir * 0.03}" rpy="0 0 1.472622"/>
+        <geometry><box size="0.01 0.020616 0.2"/></geometry></collision>
+      <visual><origin xyz="-0.008748 0.088820 ${z_dir * 0.03}" rpy="0 0 1.668971"/>
+        <geometry><box size="0.01 0.020616 0.2"/></geometry>
+        <material name="${prefix}_seg_mat"><color rgba="${seg_rgba}"/></material></visual>
+      <collision><origin xyz="-0.008748 0.088820 ${z_dir * 0.03}" rpy="0 0 1.668971"/>
+        <geometry><box size="0.01 0.020616 0.2"/></geometry></collision>
+      <visual><origin xyz="-0.025908 0.085407 ${z_dir * 0.03}" rpy="0 0 1.865321"/>
+        <geometry><box size="0.01 0.020616 0.2"/></geometry>
+        <material name="${prefix}_seg_mat"><color rgba="${seg_rgba}"/></material></visual>
+      <collision><origin xyz="-0.025908 0.085407 ${z_dir * 0.03}" rpy="0 0 1.865321"/>
+        <geometry><box size="0.01 0.020616 0.2"/></geometry></collision>
+      <visual><origin xyz="-0.042072 0.078712 ${z_dir * 0.03}" rpy="0 0 2.061670"/>
+        <geometry><box size="0.01 0.020616 0.2"/></geometry>
+        <material name="${prefix}_seg_mat"><color rgba="${seg_rgba}"/></material></visual>
+      <collision><origin xyz="-0.042072 0.078712 ${z_dir * 0.03}" rpy="0 0 2.061670"/>
+        <geometry><box size="0.01 0.020616 0.2"/></geometry></collision>
+      <visual><origin xyz="-0.056619 0.068991 ${z_dir * 0.03}" rpy="0 0 2.258020"/>
+        <geometry><box size="0.01 0.020616 0.2"/></geometry>
+        <material name="${prefix}_seg_mat"><color rgba="${seg_rgba}"/></material></visual>
+      <collision><origin xyz="-0.056619 0.068991 ${z_dir * 0.03}" rpy="0 0 2.258020"/>
+        <geometry><box size="0.01 0.020616 0.2"/></geometry></collision>
+      <visual><origin xyz="-0.068991 0.056619 ${z_dir * 0.03}" rpy="0 0 2.454369"/>
+        <geometry><box size="0.01 0.020616 0.2"/></geometry>
+        <material name="${prefix}_seg_mat"><color rgba="${seg_rgba}"/></material></visual>
+      <collision><origin xyz="-0.068991 0.056619 ${z_dir * 0.03}" rpy="0 0 2.454369"/>
+        <geometry><box size="0.01 0.020616 0.2"/></geometry></collision>
+      <visual><origin xyz="-0.078712 0.042072 ${z_dir * 0.03}" rpy="0 0 2.650719"/>
+        <geometry><box size="0.01 0.020616 0.2"/></geometry>
+        <material name="${prefix}_seg_mat"><color rgba="${seg_rgba}"/></material></visual>
+      <collision><origin xyz="-0.078712 0.042072 ${z_dir * 0.03}" rpy="0 0 2.650719"/>
+        <geometry><box size="0.01 0.020616 0.2"/></geometry></collision>
+      <visual><origin xyz="-0.085407 0.025908 ${z_dir * 0.03}" rpy="0 0 2.847068"/>
+        <geometry><box size="0.01 0.020616 0.2"/></geometry>
+        <material name="${prefix}_seg_mat"><color rgba="${seg_rgba}"/></material></visual>
+      <collision><origin xyz="-0.085407 0.025908 ${z_dir * 0.03}" rpy="0 0 2.847068"/>
+        <geometry><box size="0.01 0.020616 0.2"/></geometry></collision>
+      <visual><origin xyz="-0.088820 0.008748 ${z_dir * 0.03}" rpy="0 0 3.043418"/>
+        <geometry><box size="0.01 0.020616 0.2"/></geometry>
+        <material name="${prefix}_seg_mat"><color rgba="${seg_rgba}"/></material></visual>
+      <collision><origin xyz="-0.088820 0.008748 ${z_dir * 0.03}" rpy="0 0 3.043418"/>
+        <geometry><box size="0.01 0.020616 0.2"/></geometry></collision>
+      <visual><origin xyz="-0.088820 -0.008748 ${z_dir * 0.03}" rpy="0 0 3.239767"/>
+        <geometry><box size="0.01 0.020616 0.2"/></geometry>
+        <material name="${prefix}_seg_mat"><color rgba="${seg_rgba}"/></material></visual>
+      <collision><origin xyz="-0.088820 -0.008748 ${z_dir * 0.03}" rpy="0 0 3.239767"/>
+        <geometry><box size="0.01 0.020616 0.2"/></geometry></collision>
+      <visual><origin xyz="-0.085407 -0.025908 ${z_dir * 0.03}" rpy="0 0 3.436117"/>
+        <geometry><box size="0.01 0.020616 0.2"/></geometry>
+        <material name="${prefix}_seg_mat"><color rgba="${seg_rgba}"/></material></visual>
+      <collision><origin xyz="-0.085407 -0.025908 ${z_dir * 0.03}" rpy="0 0 3.436117"/>
+        <geometry><box size="0.01 0.020616 0.2"/></geometry></collision>
+      <visual><origin xyz="-0.078712 -0.042072 ${z_dir * 0.03}" rpy="0 0 3.632467"/>
+        <geometry><box size="0.01 0.020616 0.2"/></geometry>
+        <material name="${prefix}_seg_mat"><color rgba="${seg_rgba}"/></material></visual>
+      <collision><origin xyz="-0.078712 -0.042072 ${z_dir * 0.03}" rpy="0 0 3.632467"/>
+        <geometry><box size="0.01 0.020616 0.2"/></geometry></collision>
+      <visual><origin xyz="-0.068991 -0.056619 ${z_dir * 0.03}" rpy="0 0 3.828816"/>
+        <geometry><box size="0.01 0.020616 0.2"/></geometry>
+        <material name="${prefix}_seg_mat"><color rgba="${seg_rgba}"/></material></visual>
+      <collision><origin xyz="-0.068991 -0.056619 ${z_dir * 0.03}" rpy="0 0 3.828816"/>
+        <geometry><box size="0.01 0.020616 0.2"/></geometry></collision>
+      <visual><origin xyz="-0.056619 -0.068991 ${z_dir * 0.03}" rpy="0 0 4.025166"/>
+        <geometry><box size="0.01 0.020616 0.2"/></geometry>
+        <material name="${prefix}_seg_mat"><color rgba="${seg_rgba}"/></material></visual>
+      <collision><origin xyz="-0.056619 -0.068991 ${z_dir * 0.03}" rpy="0 0 4.025166"/>
+        <geometry><box size="0.01 0.020616 0.2"/></geometry></collision>
+      <visual><origin xyz="-0.042072 -0.078712 ${z_dir * 0.03}" rpy="0 0 4.221515"/>
+        <geometry><box size="0.01 0.020616 0.2"/></geometry>
+        <material name="${prefix}_seg_mat"><color rgba="${seg_rgba}"/></material></visual>
+      <collision><origin xyz="-0.042072 -0.078712 ${z_dir * 0.03}" rpy="0 0 4.221515"/>
+        <geometry><box size="0.01 0.020616 0.2"/></geometry></collision>
+      <visual><origin xyz="-0.025908 -0.085407 ${z_dir * 0.03}" rpy="0 0 4.417865"/>
+        <geometry><box size="0.01 0.020616 0.2"/></geometry>
+        <material name="${prefix}_seg_mat"><color rgba="${seg_rgba}"/></material></visual>
+      <collision><origin xyz="-0.025908 -0.085407 ${z_dir * 0.03}" rpy="0 0 4.417865"/>
+        <geometry><box size="0.01 0.020616 0.2"/></geometry></collision>
+      <visual><origin xyz="-0.008748 -0.088820 ${z_dir * 0.03}" rpy="0 0 4.614214"/>
+        <geometry><box size="0.01 0.020616 0.2"/></geometry>
+        <material name="${prefix}_seg_mat"><color rgba="${seg_rgba}"/></material></visual>
+      <collision><origin xyz="-0.008748 -0.088820 ${z_dir * 0.03}" rpy="0 0 4.614214"/>
+        <geometry><box size="0.01 0.020616 0.2"/></geometry></collision>
+      <visual><origin xyz="0.008748 -0.088820 ${z_dir * 0.03}" rpy="0 0 4.810564"/>
+        <geometry><box size="0.01 0.020616 0.2"/></geometry>
+        <material name="${prefix}_seg_mat"><color rgba="${seg_rgba}"/></material></visual>
+      <collision><origin xyz="0.008748 -0.088820 ${z_dir * 0.03}" rpy="0 0 4.810564"/>
+        <geometry><box size="0.01 0.020616 0.2"/></geometry></collision>
+      <visual><origin xyz="0.025908 -0.085407 ${z_dir * 0.03}" rpy="0 0 5.006913"/>
+        <geometry><box size="0.01 0.020616 0.2"/></geometry>
+        <material name="${prefix}_seg_mat"><color rgba="${seg_rgba}"/></material></visual>
+      <collision><origin xyz="0.025908 -0.085407 ${z_dir * 0.03}" rpy="0 0 5.006913"/>
+        <geometry><box size="0.01 0.020616 0.2"/></geometry></collision>
+      <visual><origin xyz="0.042072 -0.078712 ${z_dir * 0.03}" rpy="0 0 5.203263"/>
+        <geometry><box size="0.01 0.020616 0.2"/></geometry>
+        <material name="${prefix}_seg_mat"><color rgba="${seg_rgba}"/></material></visual>
+      <collision><origin xyz="0.042072 -0.078712 ${z_dir * 0.03}" rpy="0 0 5.203263"/>
+        <geometry><box size="0.01 0.020616 0.2"/></geometry></collision>
+      <visual><origin xyz="0.056619 -0.068991 ${z_dir * 0.03}" rpy="0 0 5.399612"/>
+        <geometry><box size="0.01 0.020616 0.2"/></geometry>
+        <material name="${prefix}_seg_mat"><color rgba="${seg_rgba}"/></material></visual>
+      <collision><origin xyz="0.056619 -0.068991 ${z_dir * 0.03}" rpy="0 0 5.399612"/>
+        <geometry><box size="0.01 0.020616 0.2"/></geometry></collision>
+      <visual><origin xyz="0.068991 -0.056619 ${z_dir * 0.03}" rpy="0 0 5.595962"/>
+        <geometry><box size="0.01 0.020616 0.2"/></geometry>
+        <material name="${prefix}_seg_mat"><color rgba="${seg_rgba}"/></material></visual>
+      <collision><origin xyz="0.068991 -0.056619 ${z_dir * 0.03}" rpy="0 0 5.595962"/>
+        <geometry><box size="0.01 0.020616 0.2"/></geometry></collision>
+      <visual><origin xyz="0.078712 -0.042072 ${z_dir * 0.03}" rpy="0 0 5.792311"/>
+        <geometry><box size="0.01 0.020616 0.2"/></geometry>
+        <material name="${prefix}_seg_mat"><color rgba="${seg_rgba}"/></material></visual>
+      <collision><origin xyz="0.078712 -0.042072 ${z_dir * 0.03}" rpy="0 0 5.792311"/>
+        <geometry><box size="0.01 0.020616 0.2"/></geometry></collision>
+      <visual><origin xyz="0.085407 -0.025908 ${z_dir * 0.03}" rpy="0 0 5.988661"/>
+        <geometry><box size="0.01 0.020616 0.2"/></geometry>
+        <material name="${prefix}_seg_mat"><color rgba="${seg_rgba}"/></material></visual>
+      <collision><origin xyz="0.085407 -0.025908 ${z_dir * 0.03}" rpy="0 0 5.988661"/>
+        <geometry><box size="0.01 0.020616 0.2"/></geometry></collision>
+      <visual><origin xyz="0.088820 -0.008748 ${z_dir * 0.03}" rpy="0 0 6.185011"/>
+        <geometry><box size="0.01 0.020616 0.2"/></geometry>
+        <material name="${prefix}_seg_mat"><color rgba="${seg_rgba}"/></material></visual>
+      <collision><origin xyz="0.088820 -0.008748 ${z_dir * 0.03}" rpy="0 0 6.185011"/>
+        <geometry><box size="0.01 0.020616 0.2"/></geometry></collision>
     </link>
-    <!-- Cup wall -X -->
-    <link name="${prefix}_cup_wall_x_minus">
-      <visual>
-        <origin xyz="0 0 0" rpy="0 0 0"/>
-        <geometry>
-          <box size="0.005 0.1 0.1"/>
-        </geometry>
-        <material name="wood"/>
-      </visual>
-      <collision>
-        <origin xyz="0 0 0" rpy="0 0 0"/>
-        <geometry>
-          <box size="0.005 0.1 0.1"/>
-        </geometry>
-      </collision>
-      <inertial>
-        <origin xyz="0 0 0" rpy="0 0 0"/>
-        <mass value="0.015"/>
-        <inertia ixx="0.0001" ixy="0.0" ixz="0.0"
-                 iyy="0.0001" iyz="0.0"
-                 izz="0.00001"/>
-      </inertial>
-    </link>
-    <!-- Cup wall +Y -->
-    <link name="${prefix}_cup_wall_y_plus">
-      <visual>
-        <origin xyz="0 0 0" rpy="0 0 0"/>
-        <geometry>
-          <box size="0.1 0.005 0.1"/>
-        </geometry>
-        <material name="wood"/>
-      </visual>
-      <collision>
-        <origin xyz="0 0 0" rpy="0 0 0"/>
-        <geometry>
-          <box size="0.1 0.005 0.1"/>
-        </geometry>
-      </collision>
-      <inertial>
-        <origin xyz="0 0 0" rpy="0 0 0"/>
-        <mass value="0.015"/>
-        <inertia ixx="0.0001" ixy="0.0" ixz="0.0"
-                 iyy="0.00001" iyz="0.0"
-                 izz="0.0001"/>
-      </inertial>
-    </link>
-    <!-- Cup wall -Y -->
-    <link name="${prefix}_cup_wall_y_minus">
-      <visual>
-        <origin xyz="0 0 0" rpy="0 0 0"/>
-        <geometry>
-          <box size="0.1 0.005 0.1"/>
-        </geometry>
-        <material name="wood"/>
-      </visual>
-      <collision>
-        <origin xyz="0 0 0" rpy="0 0 0"/>
-        <geometry>
-          <box size="0.1 0.005 0.1"/>
-        </geometry>
-      </collision>
-      <inertial>
-        <origin xyz="0 0 0" rpy="0 0 0"/>
-        <mass value="0.015"/>
-        <inertia ixx="0.0001" ixy="0.0" ixz="0.0"
-                 iyy="0.00001" iyz="0.0"
-                 izz="0.0001"/>
-      </inertial>
-    </link>
-    <!-- Mount cup pole to parent (end effector) -->
-    <joint name="${prefix}_cup_mount_joint" type="fixed">
+    <!-- Fixed joint attaching the cup to its parent link -->
+    <joint name="${prefix}_cup_joint" type="fixed">
       <xacro:insert_block name="origin"/>
       <parent link="${parent}"/>
-      <child link="${prefix}_cup_pole"/>
-    </joint>
-    <!-- Attach cup bottom to pole (at z=0.08, centered in pole) -->
-    <joint name="${prefix}_cup_bottom_joint" type="fixed">
-      <origin xyz="0 0 0.08" rpy="0 0 0"/>
-      <parent link="${prefix}_cup_pole"/>
-      <child link="${prefix}_cup_bottom"/>
-    </joint>
-    <!-- Attach cup walls (centered at z=0.18, which is middle of 0.2m wall height) -->
-    <joint name="${prefix}_cup_wall_x_plus_joint" type="fixed">
-      <origin xyz="0.060 0 0.12" rpy="0 0 0"/>
-      <parent link="${prefix}_cup_pole"/>
-      <child link="${prefix}_cup_wall_x_plus"/>
-    </joint>
-    <joint name="${prefix}_cup_wall_x_minus_joint" type="fixed">
-      <origin xyz="-0.060 0 0.12" rpy="0 0 0"/>
-      <parent link="${prefix}_cup_pole"/>
-      <child link="${prefix}_cup_wall_x_minus"/>
-    </joint>
-    <joint name="${prefix}_cup_wall_y_plus_joint" type="fixed">
-      <origin xyz="0 0.060 0.12" rpy="0 0 0"/>
-      <parent link="${prefix}_cup_pole"/>
-      <child link="${prefix}_cup_wall_y_plus"/>
-    </joint>
-    <joint name="${prefix}_cup_wall_y_minus_joint" type="fixed">
-      <origin xyz="0 -0.060 0.12" rpy="0 0 0"/>
-      <parent link="${prefix}_cup_pole"/>
-      <child link="${prefix}_cup_wall_y_minus"/>
+      <child link="${prefix}_cup"/>
     </joint>
   </xacro:macro>
