Commit message: final

File: bimanual_ws/src/bimanualrobot_ros2/bimanualrobot_description/urdf/robots/bimanualrobot.urdf (robot description, URDF)
Before this commit: robot bimanualrobot, 23 links, 22 joints
Links:
- link leftarm_forearm_link: geometry collision mesh filename=file:///home/asurite.ad.asu.edu/troisin/Documents/robot/bim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; visual mesh filename=file:///home/asurite.ad.asu.edu/troisin/Documents/robot/bim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 scale=0.001 0.001 0.001
- link leftarm_shoulder_link: geometry collision box size=0.054 0.054 0.126; visual mesh filename=file:///home/asurite.ad.asu.edu/troisin/Documents/robot/bim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 scale=0.001 0.001 0.001
- link leftarm_upper_arm_link: geometry collision box size=0.06 0.14 0.06; visual mesh filename=file:///home/asurite.ad.asu.edu/troisin/Documents/robot/bim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 scale=0.001 0.001 0.001
- link leftarm_wrist_1_link: geometry collision mesh filename=file:///home/asurite.ad.asu.edu/troisin/Documents/robot/bim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; visual mesh filename=file:///home/asurite.ad.asu.edu/troisin/Documents/robot/bim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 scale=0.001 0.001 0.001
- link leftarm_wrist_2_link: geometry collision box size=0.048 0.09 0.048; visual mesh filename=file:///home/asurite.ad.asu.edu/troisin/Documents/robot/bim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 scale=0.001 0.001 0.001
- link leftarm_wrist_3_link: geometry collision mesh filename=file:///home/asurite.ad.asu.edu/troisin/Documents/robot/bim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; visual mesh filename=file:///home/asurite.ad.asu.edu/troisin/Documents/robot/bim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 scale=0.001 0.001 0.001
- link rightarm_forearm_link: geometry collision mesh filename=file:///home/asurite.ad.asu.edu/troisin/Documents/robot/bim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; visual mesh filename=file:///home/asurite.ad.asu.edu/troisin/Documents/robot/bim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 scale=0.001 0.001 0.001
- link rightarm_shoulder_link: geometry collision box size=0.054 0.054 0.126; visual mesh filename=file:///home/asurite.ad.asu.edu/troisin/Documents/robot/bim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 scale=0.001 0.001 0.001
- link rightarm_upper_arm_link: geometry collision box size=0.06 0.14 0.06; visual mesh filename=file:///home/asurite.ad.asu.edu/troisin/Documents/robot/bim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 scale=0.001 0.001 0.001
- link rightarm_wrist_1_link: geometry collision mesh filename=file:///home/asurite.ad.asu.edu/troisin/Documents/robot/bim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; visual mesh filename=file:///home/asurite.ad.asu.edu/troisin/Documents/robot/bim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 scale=0.001 0.001 0.001
- link rightarm_wrist_2_link: geometry collision box size=0.048 0.09 0.048; visual mesh filename=file:///home/asurite.ad.asu.edu/troisin/Documents/robot/bim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 scale=0.001 0.001 0.001
- link rightarm_wrist_3_link: geometry collision mesh filename=file:///home/asurite.ad.asu.edu/troisin/Documents/robot/bim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; visual mesh filename=file:///home/asurite.ad.asu.edu/troisin/Documents/robot/bim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 scale=0.001 0.001 0.001
- link stand_link: geometry collision mesh filename=file:///home/asurite.ad.asu.edu/troisin/Documents/robot/bim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; visual mesh filename=file:///home/asurite.ad.asu.edu/troisin/Documents/robot/bim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

File: bimanual_ws/src/bimanualrobot_ros2/bimanualrobot_description/urdf/robots/bimanualrobot.urdf.xacro (robot description, xacro)
@@ -88,9 +88,9 @@
     <!-- Left cup and ball - matching MuJoCo orientation (1.5707963 0 0) -->
     <xacro:cup_and_ball prefix="leftarm" parent="leftarm_ee_link">
-      <origin xyz="0 0.15 0.09" rpy="1.5707963 0 0" />
+      <origin xyz="0 0.01 0.09" rpy="1.5707963 0 0" />
     </xacro:cup_and_ball>
     <!-- Right cup and ball - ADD PI rotation to compensate for arm orientation difference -->
     <xacro:cup_and_ball prefix="rightarm" parent="rightarm_ee_link">
-      <origin xyz="0 -0.15 0.09" rpy="1.5707963 0 ${pi}" />
+      <origin xyz="0 -0.01 0.09" rpy="1.5707963 0 ${pi}" />
     </xacro:cup_and_ball>
   </xacro:if>
